Commit message: Add FSR sensors
Edited model file to include FSR sensors on each feet.

File: urdf/darwin.urdf (robot description, URDF)
Before this commit: robot darwinOP, 31 links, 30 joints
Links:
- added link Left_FSR_BL_frame, mass 0.08057; collision cylinder length=0.005 radius=0.005; visual cylinder length=0.005 radius=0.005
- added link Left_FSR_BR_frame, mass 0.08057; collision cylinder length=0.005 radius=0.005; visual cylinder length=0.005 radius=0.005
- added link Left_FSR_FL_frame, mass 0.08057; collision cylinder length=0.005 radius=0.005; visual cylinder length=0.005 radius=0.005
- added link Left_FSR_FR_frame, mass 0.08057; collision cylinder length=0.005 radius=0.005; visual cylinder length=0.005 radius=0.005
- added link Right_FSR_BL_frame, mass 0.08057; collision cylinder length=0.005 radius=0.005; visual cylinder length=0.005 radius=0.005
- added link Right_FSR_BR_frame, mass 0.08057; collision cylinder length=0.005 radius=0.005; visual cylinder length=0.005 radius=0.005
- added link Right_FSR_FL_frame, mass 0.08057; collision cylinder length=0.005 radius=0.005; visual cylinder length=0.005 radius=0.005
- added link Right_FSR_FR_frame, mass 0.08057; collision cylinder length=0.005 radius=0.005; visual cylinder length=0.005 radius=0.005
Joints:
- added joint Left_FSR_BL_fixedjoint: type fixed, parent MP_ANKLE2_L, child Left_FSR_BL_frame, origin xyz=-0.0335 -0.0355 -0.041 rpy=0 0 0, axis 0 0 0
- added joint Left_FSR_BR_fixedjoint: type fixed, parent MP_ANKLE2_L, child Left_FSR_BR_frame, origin xyz=-0.0335 0.0145 -0.041 rpy=0 0 0, axis 0 0 0
- added joint Left_FSR_FL_fixedjoint: type fixed, parent MP_ANKLE2_L, child Left_FSR_FL_frame, origin xyz=-0.0335 -0.0355 0.041 rpy=0 0 0, axis 0 0 0
- added joint Left_FSR_FR_fixedjoint: type fixed, parent MP_ANKLE2_L, child Left_FSR_FR_frame, origin xyz=-0.0335 0.0145 0.041 rpy=0 0 0, axis 0 0 0
- added joint Right_FSR_BL_fixedjoint: type fixed, parent MP_ANKLE2_R, child Right_FSR_BL_frame, origin xyz=0.0335 0.0145 -0.041 rpy=0 0 0, axis 0 0 0
- added joint Right_FSR_BR_fixedjoint: type fixed, parent MP_ANKLE2_R, child Right_FSR_BR_frame, origin xyz=0.0335 -0.0355 -0.041 rpy=0 0 0, axis 0 0 0
- added joint Right_FSR_FL_fixedjoint: type fixed, parent MP_ANKLE2_R, child Right_FSR_FL_frame, origin xyz=0.0335 0.0145 0.041 rpy=0 0 0, axis 0 0 0
- added joint Right_FSR_FR_fixedjoint: type fixed, parent MP_ANKLE2_R, child Right_FSR_FR_frame, origin xyz=0.0335 -0.0355 0.041 rpy=0 0 0, axis 0 0 0

Commit message: Replaced cylindrical FSR sensors by cubic FSR sensors
Adjusted inertial matrix for cubic shape.

Fixed missing '<gazebo>' tags on IMU sensor definition.

File: urdf/darwin.urdf (robot description, URDF)
Before this commit: robot darwinOP, 39 links, 38 joints
Links:
- link Left_FSR_BL_frame: geometry collision box size=0.01 0.01 0.01; visual box size=0.01 0.01 0.01
- link Left_FSR_BR_frame: geometry collision box size=0.01 0.01 0.01; visual box size=0.01 0.01 0.01
- link Left_FSR_FL_frame: geometry collision box size=0.01 0.01 0.01; visual box size=0.01 0.01 0.01
- link Left_FSR_FR_frame: geometry collision box size=0.01 0.01 0.01; visual box size=0.01 0.01 0.01
- link Right_FSR_BL_frame: geometry collision box size=0.01 0.01 0.01; visual box size=0.01 0.01 0.01
- link Right_FSR_BR_frame: geometry collision box size=0.01 0.01 0.01; visual box size=0.01 0.01 0.01
- link Right_FSR_FL_frame: geometry collision box size=0.01 0.01 0.01; visual box size=0.01 0.01 0.01
- link Right_FSR_FR_frame: geometry collision box size=0.01 0.01 0.01; visual box size=0.01 0.01 0.01

Commit message: Update Joint Limit Interface values on URDF file
Replace the default joint limit values [-150, 150] for the leg joints on
the URDF model file with the values supplied in:
 https://citeseerx.ist.psu.edu/viewdoc/download?doi=10.1.1.822.6324&rep=rep1&type=pdf

File: urdf/darwin.urdf (robot description, URDF)
Before this commit: robot darwinOP, 39 links, 38 joints
Joints:
- joint j_ankle1_l: limit lower=-2.6179939 upper=2.6179939 effort=10 velocity=5.6548668 -> lower=-1.047197551 upper=1.047197551 effort=10 velocity=5.6548668
- joint j_ankle1_r: limit lower=-2.6179939 upper=2.6179939 effort=10 velocity=5.6548668 -> lower=-1.047197551 upper=1.047197551 effort=10 velocity=5.6548668
- joint j_ankle2_l: limit lower=-2.6179939 upper=2.6179939 effort=10 velocity=5.6548668 -> lower=-0.5235987756 upper=1.047197551 effort=10 velocity=5.6548668
- joint j_ankle2_r: limit lower=-2.6179939 upper=2.6179939 effort=10 velocity=5.6548668 -> lower=-0.5235987756 upper=1.047197551 effort=10 velocity=5.6548668
- joint j_pelvis_l: limit lower=-2.6179939 upper=2.6179939 effort=10 velocity=5.6548668 -> lower=-0.7853981634 upper=2.617993878 effort=10 velocity=5.6548668
- joint j_pelvis_r: limit lower=-2.6179939 upper=2.6179939 effort=10 velocity=5.6548668 -> lower=-2.617993878 upper=0.7853981634 effort=10 velocity=5.6548668
- joint j_thigh1_l: limit lower=-2.6179939 upper=2.6179939 effort=10 velocity=5.6548668 -> lower=-1.047197551 upper=0.0000 effort=10 velocity=5.6548668
- joint j_thigh1_r: limit lower=-2.6179939 upper=2.6179939 effort=10 velocity=5.6548668 -> lower=0.0000 upper=1.047197551 effort=10 velocity=5.6548668
- joint j_thigh2_l: limit lower=-2.6179939 upper=2.6179939 effort=10 velocity=5.6548668 -> lower=-0.5235987756 upper=1.745329252 effort=10 velocity=5.6548668
- joint j_thigh2_r: limit lower=-2.6179939 upper=2.6179939 effort=10 velocity=5.6548668 -> lower=-1.745329252 upper=0.5235987756 effort=10 velocity=5.6548668
- joint j_tibia_l: limit lower=-2.6179939 upper=2.6179939 effort=10 velocity=5.6548668 -> lower=-2.2689280276 upper=0.0000 effort=10 velocity=5.6548668
- joint j_tibia_r: limit lower=-2.6179939 upper=2.6179939 effort=10 velocity=5.6548668 -> lower=0.0000 upper=2.2689280276 effort=10 velocity=5.6548668

Commit message: Add FSR sensors to feet and correct left pelvis link

File: urdf/darwin.urdf (robot description, URDF)
Before this commit: robot darwinOP, 39 links, 38 joints
Links:
- link MP_PELVIS_L: mass 0.167 -> 0.197
Joints:
- joint j_ankle1_l: limit lower=-1.047197551 upper=1.047197551 effort=10 velocity=5.6548668 -> lower=-2.6179939 upper=2.6179939 effort=10 velocity=5.6548668
- joint j_ankle1_r: limit lower=-1.047197551 upper=1.047197551 effort=10 velocity=5.6548668 -> lower=-2.6179939 upper=2.6179939 effort=10 velocity=5.6548668
- joint j_ankle2_l: limit lower=-0.5235987756 upper=1.047197551 effort=10 velocity=5.6548668 -> lower=-2.6179939 upper=2.6179939 effort=10 velocity=5.6548668
- joint j_ankle2_r: limit lower=-0.5235987756 upper=1.047197551 effort=10 velocity=5.6548668 -> lower=-2.6179939 upper=2.6179939 effort=10 velocity=5.6548668
- joint j_pelvis_l: limit lower=-0.7853981634 upper=2.617993878 effort=10 velocity=5.6548668 -> lower=-2.6179939 upper=2.6179939 effort=10 velocity=5.6548668
- joint j_pelvis_r: limit lower=-2.617993878 upper=0.7853981634 effort=10 velocity=5.6548668 -> lower=-2.6179939 upper=2.6179939 effort=10 velocity=5.6548668
- joint j_thigh1_l: limit lower=-1.047197551 upper=0.0000 effort=10 velocity=5.6548668 -> lower=-2.6179939 upper=2.6179939 effort=10 velocity=5.6548668
- joint j_thigh1_r: limit lower=0.0000 upper=1.047197551 effort=10 velocity=5.6548668 -> lower=-2.6179939 upper=2.6179939 effort=10 velocity=5.6548668
- joint j_thigh2_l: limit lower=-0.5235987756 upper=1.745329252 effort=10 velocity=5.6548668 -> lower=-2.6179939 upper=2.6179939 effort=10 velocity=5.6548668
- joint j_thigh2_r: limit lower=-1.745329252 upper=0.5235987756 effort=10 velocity=5.6548668 -> lower=-2.6179939 upper=2.6179939 effort=10 velocity=5.6548668
- joint j_tibia_l: limit lower=-2.2689280276 upper=0.0000 effort=10 velocity=5.6548668 -> lower=-2.6179939 upper=2.6179939 effort=10 velocity=5.6548668
- joint j_tibia_r: limit lower=0.0000 upper=2.2689280276 effort=10 velocity=5.6548668 -> lower=-2.6179939 upper=2.6179939 effort=10 velocity=5.6548668
